Commit message: Complete simulation

File: urdf/camera.xacro (robot description, xacro)
@@ -20,4 +20,7 @@
                     <box size="${length} ${width} ${height}"/>
                 </geometry>
+                <material name="yellow">
+                    <color rgba="1 1 0 1"/>
+                  </material>
             </visual>
             <collision>
@@ -29,9 +32,43 @@
                 </geometry>
             </collision>
-            <material name="Red">
-                <color rgba="1.0 0.0 0.0 1.0"/>
-            </material>
             <xacro:inertial_matrix mass="${mass}"/>
         </link>
+        <gazebo reference ="${link_name}">
+            <material>Gazebo/Yellow</material>
+            <sensor type="camera" name="camera_1">
+                <update_rate>30.0</update_rate>
+                <camera name="camera">
+                  <horizontal_fov>1.3962634</horizontal_fov>
+                  <image>
+                    <width>400</width>
+                    <height>400</height>
+                    <format>R8G8B8</format>
+                  </image>
+                  <clip>
+                    <near>0.02</near>
+                    <far>300</far>
+                  </clip>
+                  <noise>
+                    <type>gaussian</type>
+                    <mean>0.0</mean>
+                    <stddev>0.007</stddev>
+                  </noise>
+                </camera>
+                <plugin name="camera_controller" filename="libgazebo_ros_camera.so">
+                  <alwaysOn>true</alwaysOn>
+                  <updateRate>0.0</updateRate>
+                  <cameraName>camera</cameraName>
+                  <imageTopicName>image_raw</imageTopicName>
+                  <cameraInfoTopicName>camera_info</cameraInfoTopicName>
+                  <frameName>camera_link</frameName>
+                  <hackBaseline>0.07</hackBaseline>
+                  <distortionK1>0.0</distortionK1>
+                  <distortionK2>0.0</distortionK2>
+                  <distortionK3>0.0</distortionK3>
+                  <distortionT1>0.0</distortionT1>
+                  <distortionT2>0.0</distortionT2>
+                </plugin>
+              </sensor>
+          </gazebo>
 </xacro:macro>
 </robot>

File: urdf/common_macro.xacro (robot description, xacro)
@@ -54,12 +54,24 @@
     <transmission name="${joint_name}_rotation_trans">
         <type>transmission_interface/SimpleTransmission</type>
-        <actuator name="${joint_name}_rotation_motor">
-            <hardwareInterface>EffortJointInterface</hardwareInterface>
+        <actuator name="${joint_name}_motor">
             <mechanicalReduction>1</mechanicalReduction>
         </actuator>
-            <joint name="${joint_name}">
-            <hardwareInterface>VelocityJointInterface</hardwareInterface>
+        <joint name="${joint_name}">
+            <hardwareInterface>hardware_interface/VelocityJointInterface</hardwareInterface>
         </joint>
     </transmission>
 </xacro:macro>
+<!-- *********************************************************************** -->
+<!--Fixed cilinder block-->
+<xacro:macro name="Fixed_rotation_block" params="joint_name">
+    <transmission name="${joint_name}_fixed_rotation">
+        <type>transmission_interface/SimpleTransmission</type>
+        <actuator name="$${joint_name}_motor">
+          <mechanicalReduction>1</mechanicalReduction>
+        </actuator>
+        <joint name="${joint_name}">
+          <hardwareInterface>hardware_interface/PositionJointInterface</hardwareInterface>
+        </joint>
+      </transmission>
+</xacro:macro>
 </robot>

File: urdf/control_block.xacro (robot description, xacro)
@@ -20,4 +20,7 @@
                 <box size="${length} ${width} ${height}"/>
             </geometry>
+            <material name="Red">
+                <color rgba="1.0 0.0 0.0 1.0"/>
+            </material>
         </visual>
         <collision>
@@ -29,9 +32,9 @@
             </geometry>
         </collision>
-        <material name="Red">
-            <color rgba="1.0 0.0 0.0 1.0"/>
-        </material>
         <xacro:inertial_matrix mass="${mass}"/>
     </link>
+    <gazebo reference ="${link_name}">
+        <material>Gazebo/Red</material>
+     </gazebo>
 </xacro:macro>
 </robot>

File: urdf/corpus.xacro (robot description, xacro)
@@ -20,4 +20,7 @@
                 <box size="${length} ${width} ${height}"/>
             </geometry>
+            <material name="Blue">
+                <color rgba="0.0 0.0 1.0 1.0"/>
+            </material>
         </visual>
         <collision>
@@ -29,9 +32,9 @@
             </geometry>
         </collision>
-        <material name="Blue">
-            <color rgba="0.0 0.0 1.0 1.0"/>
-        </material>
         <xacro:inertial_matrix mass="${mass}"/>
     </link>
+    <gazebo reference ="${link_name}">
+        <material>Gazebo/Blue</material>
+     </gazebo>
 </xacro:macro>
 </robot>

File: urdf/main.xacro (robot description, xacro)
@@ -35,4 +35,5 @@
 <xacro:property name="wheel_width" value="0.05"/>
 <xacro:property name="wheel_mass" value="1.0"/>
+<xacro:property name="hinge_wheel_limit" value="${PI/3}"/>
 <!-- *********************************************************************** -->
 <xacro:corpus
@@ -64,9 +65,22 @@
     length="${wheel_width}"
     mass="${wheel_mass}"/>
-<!-- Add joints and transmission for 4 weel -->
+<!-- Front left weel -->
 <!-- *********************************************************************** -->
 <joint name="front_left_wheel_joint" type="continuous">
     <parent link="base_link"/>
     <child link="front_left_wheel_link"/>
+    <axis xyz="0 0 1"/>
+    <origin
+        xyz="${(corpus_len/2)-(wheel_radius)} ${(corpus_width/2)+(wheel_width/2)} 0"
+        rpy="${PI/2} 0 0" />
+    <limit effort= "30" velocity="1.0"/>
+    <dynamics damping="0.0" friction="0.0"/>
+</joint>
+<xacro:Transmission_rotation_block joint_name="front_left_wheel_joint"/>
+<!-- Front right wheel -->
+<!-- *********************************************************************** -->
+<joint name="front_right_wheel_joint" type="continuous">
+    <parent link="base_link"/>
+    <child link="front_right_wheel_link"/>
     <axis xyz="0 0 1"/>
     <origin
@@ -76,21 +90,23 @@
     <dynamics damping="0.0" friction="0.0"/>
 </joint>
-<xacro:Transmission_rotation_block joint_name="front_left_wheel_joint"/>
+<xacro:Transmission_rotation_block joint_name="front_right_wheel_joint"/>
+<!-- Back left wheel -->
 <!-- *********************************************************************** -->
-<joint name="front_right_wheel_joint" type="continuous">
+<joint name="back_left_wheel_joint" type="continuous">
     <parent link="base_link"/>
-    <child link="front_right_wheel_link"/>
+    <child link="back_left_wheel_link"/>
     <axis xyz="0 0 1"/>
     <origin
-        xyz="${(corpus_len/2)-(wheel_radius)} ${(+corpus_width/2)+(wheel_width/2)} 0"
+        xyz="${(-corpus_len/2)+(wheel_radius)} ${(+corpus_width/2)+(wheel_width/2)} 0"
         rpy="${PI/2} 0 0" />
     <limit effort= "30" velocity="1.0"/>
     <dynamics damping="0.0" friction="0.0"/>
 </joint>
-<xacro:Transmission_rotation_block joint_name="front_right_wheel_joint"/>
+<xacro:Transmission_rotation_block joint_name="back_left_wheel_joint"/>
+<!-- Back right wheel -->
 <!-- *********************************************************************** -->
-<joint name="back_left_wheel_joint" type="continuous">
+<joint name="back_right_wheel_joint" type="continuous">
     <parent link="base_link"/>
-    <child link="back_left_wheel_link"/>
+    <child link="back_right_wheel_link"/>
     <axis xyz="0 0 1"/>
     <origin
@@ -100,17 +116,6 @@
     <dynamics damping="0.0" friction="0.0"/>
 </joint>
-<xacro:Transmission_rotation_block joint_name="back_left_wheel_joint"/>
-<!-- *********************************************************************** -->
-<joint name="back_right_wheel_joint" type="continuous">
-    <parent link="base_link"/>
-    <child link="back_right_wheel_link"/>
-    <axis xyz="0 0 1"/>
-    <origin
-        xyz="${(-corpus_len/2)+(wheel_radius)} ${(corpus_width/2)+(wheel_width/2)} 0"
-        rpy="${PI/2} 0 0" />
-    <limit effort= "30" velocity="1.0"/>
-    <dynamics damping="0.0" friction="0.0"/>
-</joint>
 <xacro:Transmission_rotation_block joint_name="back_right_wheel_joint"/>
+<!-- Conntrol block -->
 <!-- *********************************************************************** -->
 <xacro:control_block
@@ -125,4 +130,5 @@
     <origin xyz="${-corpus_len/2+0.25} 0.0 ${corpus_height/2}" rpy="0 0 0"/>
 </joint>
+<!-- Camera -->
 <!-- *********************************************************************** -->
 <xacro:camera
@@ -132,13 +138,12 @@
     height="0.1"
     mass="1"/>
-<joint name="camera_joint" type="fixed">
+<joint name="camera_joint" type="continuous">
     <parent link="base_link"/>
     <child link="camera_link"/>
+    <axis xyz="0 0 1"/>
     <origin xyz="${corpus_len/2-0.05} 0.0 ${corpus_height/2}" rpy="0 0 0"/>
+    <limit effort="30" velocity="1.0"/>
 </joint>
-<!-- *********************************************************************** -->
-<!-- *********************************************************************** -->
-<!-- *********************************************************************** -->
-<!-- *********************************************************************** -->
+<xacro:Fixed_rotation_block joint_name="camera_joint"/>
 <!-- *********************************************************************** -->
 <!-- Add ROS plugin so we can interact with our robot -->
@@ -149,6 +154,2 @@
 </gazebo>
 </robot>
-<!--
-    rosrun xacro xacro main.xacro > main.urdf
-    gz sdf -p main.urdf > main.sdf
--->

File: urdf/wheel.xacro (robot description, xacro)
@@ -1,5 +1,6 @@
 <?xml version="1.0"?>
 <robot name="mobile_robot_base" xmlns:xacro="http://www.ros.org/wiki/xacro">
-<!-- <xacro:include filename="$(find mobile_robot_base_ros1)/urdf/common_macro.xacro" /> -->
+<xacro:include filename="$(find mobile_robot_base_ros1)/urdf/common_macro.xacro" />
+<!-- *********************************************************************** -->
 <xacro:macro
     name="wheel"
@@ -9,6 +10,4 @@
         length
         mass">
-    <!-- rpy (roll pitch yaw) describes rotation in radians -->
-    <!-- xyz describes translation in meters -->
     <link name="${link_name}">
         <visual>
@@ -17,4 +16,7 @@
                 <cylinder length="${length}" radius="${radius}"/>
             </geometry>
+            <material name="Black">
+                <color rgba="0.0 0.0 0.0 0.9"/>
+            </material>
         </visual>
         <collision>
@@ -24,32 +26,30 @@
             </geometry>
         </collision>
-        <material name="Black">
-            <color rgba="0.0 0.0 0.0 0.9"/>
-        </material>
-        <xacro:cylinder_inertia m="${mass}" r="${radius/3}" h="${length}"/>
+        <xacro:cylinder_inertia m="${mass}" r="${radius}" h="${length}"/>
     </link>
-    <!-- <xacro:insert_block name="joint_block" />
-    <xacro:Transmission_rotation_block joint_name="${prefix}"/> -->
-    <!-- <transmission name="${prefix}_arm_transmission">
-        <type>transmission_interface/SimpleTransmission</type>
-        <actuator name="$${prefix}_motor">
-            <hardwareInterface>EffortJointInterface</hardwareInterface>
-            <mechanicalReduction>1</mechanicalReduction>
-        </actuator>
-        <joint name="base_to_${prefix}_arm">
-            <hardwareInterface>hardware_interface/VelocityJointInterface</hardwareInterface>
-        </joint>
-    </transmission> -->
+ё
     <gazebo reference ="${link_name}">
         <material>Gazebo/Black</material>
-        <turnGravityOff>false</turnGravityOff>
      </gazebo>
-   <gazebo reference ="${link_name}">
-       <mu1 value="200.0"/>
-       <mu2 value="100.0"/>
-       <kp value="10000000.0"/>
-       <kd value= "1.0"/>
-       <material>Gazebo/Black</material>
-   </gazebo>
+</xacro:macro>
+<!-- *********************************************************************** -->
+<xacro:macro
+    name="wheel_hinge"
+    params="link_name">
+    <link name="${link_name}">
+        <visual>
+            <origin rpy="0 0 0" xyz="0 0 0"/>
+            <geometry>
+                <cylinder length="0.01" radius="0.025"/>
+            </geometry>
+            <material name="Green">
+                <color rgba="0.0 1.0 0.0 1.0"/>
+            </material>
+        </visual>
+        <xacro:cylinder_inertia m="1" r="0.1" h="0.1"/>
+    </link>
+    <gazebo reference ="${link_name}">
+        <material>Gazebo/Green</material>
+    </gazebo>
 </xacro:macro>
 </robot>
