Commit message: Собрал проект, добавил все описания и картинки

File: urdf/camera.xacro (robot description, xacro)
@@ -2,6 +2,8 @@
 <robot name="mobile_robot_base" xmlns:xacro="http://www.ros.org/wiki/xacro">
 <!-- *********************************************************************** -->
+<!-- Including a common macro -->
 <xacro:include filename="$(find mobile_robot_base_ros1)/urdf/common_macro.xacro" />
 <!-- *********************************************************************** -->
+<!-- Macro for creating a camera -->
 <xacro:macro
     name="camera"
@@ -12,63 +14,89 @@
         height
         mass">
-        <link name="${link_name}">
-            <visual>
-                <origin
-                    rpy= "0 0 0"
-                    xyz= "0 0 ${height/2}"/>
-                <geometry>
-                    <box size="${length} ${width} ${height}"/>
-                </geometry>
-                <material name="yellow">
-                    <color rgba="1 1 0 1"/>
-                  </material>
-            </visual>
-            <collision>
-                <origin
-                    rpy= "0 0 0"
-                    xyz= "0 0 ${height/2}"/>
-                <geometry>
-                    <box size="${length} ${width} ${height}"/>
-                </geometry>
-            </collision>
-            <xacro:inertial_matrix mass="${mass}"/>
-        </link>
-        <gazebo reference ="${link_name}">
-            <material>Gazebo/Yellow</material>
-            <sensor type="camera" name="camera_1">
-                <update_rate>30.0</update_rate>
-                <camera name="camera">
-                  <horizontal_fov>1.3962634</horizontal_fov>
-                  <image>
+    <!-- Creating a link for the camera object -->
+    <link name="${link_name}">
+        <!-- Visual representation of the camera -->
+        <visual>
+            <!-- Defining the position and orientation of the camera -->
+            <origin
+                rpy= "0 0 0"
+                xyz= "0 0 ${height/2}"/>
+            <!-- Geometry of the camera -->
+            <geometry>
+                <box size="${length} ${width} ${height}"/>
+            </geometry>
+            <!-- Material for visualizing the camera (yellow) -->
+            <material name="yellow">
+                <color rgba="1 1 0 1"/>
+            </material>
+        </visual>
+        <!-- Collision representation of the camera -->
+        <collision>
+            <!-- Defining the position and orientation of the camera -->
+            <origin
+                rpy= "0 0 0"
+                xyz= "0 0 ${height/2}"/>
+            <!-- Geometry of the camera -->
+            <geometry>
+                <box size="${length} ${width} ${height}"/>
+            </geometry>
+        </collision>
+        <!-- Calculation of the inertial matrix for the camera -->
+        <xacro:inertial_matrix mass="${mass}"/>
+    </link>
+    <!-- Specifying material for visualization in the Gazebo environment -->
+    <gazebo reference ="${link_name}">
+        <!-- Using material "Yellow" for visualization in Gazebo -->
+        <material>Gazebo/Yellow</material>
+        <!-- Adding a camera sensor -->
+        <sensor type="camera" name="camera_1">
+            <!-- Image update rate -->
+            <update_rate>30.0</update_rate>
+            <!-- Camera parameters -->
+            <camera name="camera">
+                <!-- Horizontal field of view -->
+                <horizontal_fov>1.3962634</horizontal_fov>
+                <!-- Image size -->
+                <image>
                     <width>400</width>
                     <height>400</height>
                     <format>R8G8B8</format>
-                  </image>
-                  <clip>
+                </image>
+                <!-- Clipping boundaries of the image -->
+                <clip>
                     <near>0.02</near>
                     <far>300</far>
-                  </clip>
-                  <noise>
+                </clip>
+                <!-- Image noise -->
+                <noise>
                     <type>gaussian</type>
                     <mean>0.0</mean>
                     <stddev>0.007</stddev>
-                  </noise>
-                </camera>
-                <plugin name="camera_controller" filename="libgazebo_ros_camera.so">
-                  <alwaysOn>true</alwaysOn>
-                  <updateRate>0.0</updateRate>
-                  <cameraName>camera</cameraName>
-                  <imageTopicName>image_raw</imageTopicName>
-                  <cameraInfoTopicName>camera_info</cameraInfoTopicName>
-                  <frameName>camera_link</frameName>
-                  <hackBaseline>0.07</hackBaseline>
-                  <distortionK1>0.0</distortionK1>
-                  <distortionK2>0.0</distortionK2>
-                  <distortionK3>0.0</distortionK3>
-                  <distortionT1>0.0</distortionT1>
-                  <distortionT2>0.0</distortionT2>
-                </plugin>
-              </sensor>
-          </gazebo>
+                </noise>
+            </camera>
+            <!-- Plugin for controlling the camera in Gazebo -->
+            <plugin name="camera_controller" filename="libgazebo_ros_camera.so">
+                <!-- Always on -->
+                <alwaysOn>true</alwaysOn>
+                <!-- Update rate (0.0 for maximum) -->
+                <updateRate>0.0</updateRate>
+                <!-- Camera name -->
+                <cameraName>camera</cameraName>
+                <!-- Image topic name -->
+                <imageTopicName>image_raw</imageTopicName>
+                <!-- Camera info topic name -->
+                <cameraInfoTopicName>camera_info</cameraInfoTopicName>
+                <!-- Camera frame name -->
+                <frameName>camera_link</frameName>
+                <!-- Distortion settings (not used) -->
+                <hackBaseline>0.07</hackBaseline>
+                <distortionK1>0.0</distortionK1>
+                <distortionK2>0.0</distortionK2>
+                <distortionK3>0.0</distortionK3>
+                <distortionT1>0.0</distortionT1>
+                <distortionT2>0.0</distortionT2>
+            </plugin>
+        </sensor>
+    </gazebo>
 </xacro:macro>
 </robot>

File: urdf/common_macro.xacro (robot description, xacro)
@@ -2,8 +2,9 @@
 <robot name="mobile_robot_base" xmlns:xacro="http://www.ros.org/wiki/xacro">
 <!-- *********************************************************************** -->
-<!-- Cilinder inertial -->
+<!-- Macro for cylinder inertial model -->
 <xacro:macro name="cylinder_inertia" params ="m r h">
   <inertial>
-   <mass value="${m}"/>
+   <mass value="${m}"/> <!-- Cylinder mass -->
+   <!-- Formulas to calculate inertia moments for cylinder -->
    <inertia ixx="${m*(3*r*r+h*h)/12}"  ixy="0.0" ixz="0.0"
             iyy="${m*(3*r*r+h*h)/12}"  iyz="0.0" izz="${m*r*r/2}"/>
@@ -11,8 +12,9 @@
 </xacro:macro>
 <!-- *********************************************************************** -->
-<!-- Base inertial matrix -->
+<!-- Macro for base inertial model -->
 <xacro:macro name= "inertial_matrix" params="mass">
   <inertial>
-    <mass value="${mass}"/>
+    <mass value="${mass}"/> <!-- Base mass -->
+    <!-- Set identity matrix for inertia moments -->
     <inertia
         ixx="1.0" ixy="0.0"
@@ -22,8 +24,10 @@
  </xacro:macro>
 <!-- *********************************************************************** -->
-<!-- <xacro:macro name="inertial_sphere" params="mass radius *origin">
+<!-- Macro for sphere inertial model -->
+<xacro:macro name="inertial_sphere" params="mass radius *origin">
     <inertial>
         <xacro:insert_block name="origin"/>
-        <mass value="${mass}" />
+        <mass value="${mass}" /> <!-- Sphere mass -->
+        <!-- Formulas to calculate inertia moments for sphere -->
         <inertia ixx="${(2/5) * mass * (radius*radius)}" ixy="0.0" ixz="0.0"
                 iyy="${(2/5) * mass * (radius*radius)}" iyz="0.0"
@@ -34,5 +38,6 @@
     <inertial>
         <xacro:insert_block name="origin"/>
-        <mass value="${mass}" />
+        <mass value="${mass}" /> <!-- Box mass -->
+        <!-- Formulas to calculate inertia moments for box -->
         <inertia ixx="${(1/12) * mass * (y*y+z*z)}" ixy="0.0" ixz="0.0"
                 iyy="${(1/12) * mass * (x*x+z*z)}" iyz="0.0"
@@ -43,12 +48,13 @@
     <inertial>
         <xacro:insert_block name="origin"/>
-        <mass value="${mass}" />
+        <mass value="${mass}" /> <!-- Cylinder mass -->
+        <!-- Formulas to calculate inertia moments for cylinder -->
         <inertia ixx="${(1/12) * mass * (3*radius*radius + length*length)}" ixy="0.0" ixz="0.0"
                 iyy="${(1/12) * mass * (3*radius*radius + length*length)}" iyz="0.0"
                 izz="${(1/2) * mass * (radius*radius)}" />
     </inertial>
-</xacro:macro> -->
+</xacro:macro>
 <!-- *********************************************************************** -->
-<!--Transmission cilinder block-->
+<!-- Transmission block for cylinder rotation -->
 <xacro:macro name="Transmission_rotation_block" params="joint_name">
     <transmission name="${joint_name}_rotation_trans">
@@ -63,5 +69,5 @@
 </xacro:macro>
 <!-- *********************************************************************** -->
-<!--Fixed cilinder block-->
+<!-- Fixed transmission block for cylinder rotation -->
 <xacro:macro name="Fixed_rotation_block" params="joint_name">
     <transmission name="${joint_name}_fixed_rotation">

File: urdf/control_block.xacro (robot description, xacro)
@@ -2,6 +2,8 @@
 <robot name="mobile_robot_base" xmlns:xacro="http://www.ros.org/wiki/xacro">
 <!-- *********************************************************************** -->
+<!-- Including a common macro -->
 <xacro:include filename="$(find mobile_robot_base_ros1)/urdf/common_macro.xacro" />
 <!-- *********************************************************************** -->
+<!-- Macro for creating a control block -->
 <xacro:macro
     name="control_block"
@@ -12,27 +14,38 @@
         height
         mass">
+    <!-- Creating a link for the control block object -->
     <link name="${link_name}">
+        <!-- Visual representation of the control block -->
         <visual>
+            <!-- Defining the position and orientation of the control block -->
             <origin
                 rpy= "0 0 0"
                 xyz= "0 0 ${height/2}"/>
+            <!-- Geometry of the control block -->
             <geometry>
                 <box size="${length} ${width} ${height}"/>
             </geometry>
+            <!-- Material for visualizing the control block (red) -->
             <material name="Red">
                 <color rgba="1.0 0.0 0.0 1.0"/>
             </material>
         </visual>
+        <!-- Collision representation of the control block -->
         <collision>
+            <!-- Defining the position and orientation of the control block -->
             <origin
                 rpy= "0 0 0"
                 xyz= "0 0 ${height/2}"/>
+            <!-- Geometry of the control block -->
             <geometry>
                 <box size="${length} ${width} ${height}"/>
             </geometry>
         </collision>
+        <!-- Calculation of the inertial matrix for the control block -->
         <xacro:inertial_matrix mass="${mass}"/>
     </link>
+    <!-- Specifying material for visualization in the Gazebo environment -->
     <gazebo reference ="${link_name}">
+        <!-- Using material "Red" for visualization in Gazebo -->
         <material>Gazebo/Red</material>
      </gazebo>

File: urdf/corpus.xacro (robot description, xacro)
@@ -2,6 +2,8 @@
 <robot name="mobile_robot_base" xmlns:xacro="http://www.ros.org/wiki/xacro">
 <!-- *********************************************************************** -->
+<!-- Including a common macro -->
 <xacro:include filename="$(find mobile_robot_base_ros1)/urdf/common_macro.xacro" />
 <!-- *********************************************************************** -->
+<!-- Macro for creating the robot body -->
 <xacro:macro
     name="corpus"
@@ -13,4 +15,5 @@
         mass">
     <link name="${link_name}">
+        <!-- Visual representation of the body -->
         <visual>
             <origin
@@ -20,8 +23,10 @@
                 <box size="${length} ${width} ${height}"/>
             </geometry>
+            <!-- Material for visualization in blue color -->
             <material name="Blue">
                 <color rgba="0.0 0.0 1.0 1.0"/>
             </material>
         </visual>
+        <!-- Collision representation of the body -->
         <collision>
              <origin
@@ -32,6 +37,8 @@
             </geometry>
         </collision>
+        <!-- Calculation of the inertial matrix for the body -->
         <xacro:inertial_matrix mass="${mass}"/>
     </link>
+    <!-- Specifying material for visualization in the Gazebo environment -->
     <gazebo reference ="${link_name}">
         <material>Gazebo/Blue</material>

File: urdf/wheel.xacro (robot description, xacro)
@@ -3,4 +3,5 @@
 <xacro:include filename="$(find mobile_robot_base_ros1)/urdf/common_macro.xacro" />
 <!-- *********************************************************************** -->
+<!-- Macro definition for creating a wheel -->
 <xacro:macro
     name="wheel"
@@ -11,4 +12,5 @@
         mass">
     <link name="${link_name}">
+        <!-- Visual representation of the wheel -->
         <visual>
             <origin rpy="0 0 0" xyz="0 0 0"/>
@@ -16,8 +18,10 @@
                 <cylinder length="${length}" radius="${radius}"/>
             </geometry>
+            <!-- Material for visualization in black color -->
             <material name="Black">
                 <color rgba="0.0 0.0 0.0 0.9"/>
             </material>
         </visual>
+        <!-- Collision representation of the wheel -->
         <collision>
             <origin rpy="0 0 0" xyz="0 0 0"/>
@@ -26,7 +30,8 @@
             </geometry>
         </collision>
+        <!-- Calculation of inertia for the wheel -->
         <xacro:cylinder_inertia m="${mass}" r="${radius}" h="${length}"/>
     </link>
-ё
+    <!-- Specifying material for visualization in Gazebo environment -->
     <gazebo reference ="${link_name}">
         <material>Gazebo/Black</material>
@@ -34,8 +39,10 @@
 </xacro:macro>
 <!-- *********************************************************************** -->
+<!-- Macro definition for creating a wheel hinge -->
 <xacro:macro
     name="wheel_hinge"
     params="link_name">
     <link name="${link_name}">
+        <!-- Visual representation of the hinge -->
         <visual>
             <origin rpy="0 0 0" xyz="0 0 0"/>
@@ -43,10 +50,13 @@
                 <cylinder length="0.01" radius="0.025"/>
             </geometry>
+            <!-- Material for visualization in green color -->
             <material name="Green">
                 <color rgba="0.0 1.0 0.0 1.0"/>
             </material>
         </visual>
+        <!-- Calculation of inertia for the hinge -->
         <xacro:cylinder_inertia m="1" r="0.1" h="0.1"/>
     </link>
+    <!-- Specifying material for visualization in Gazebo environment -->
     <gazebo reference ="${link_name}">
         <material>Gazebo/Green</material>
